File: kicad/project one dac.sch (KiCad schematic (older format))
At the start: 12 parts

Commit message: Forgot to add annotation
Parts:
- gave numbers to parts that had none: 12
Changed lines of the file:
@@
 $EndDescr
 $Comp
-L PCM5100 U?
+L PCM5100 U501
 U 1 1 53676BCE
 P 5950 3400
-F 0 "U?" H 5550 3950 60  0000 C CNN
+F 0 "U501" H 5550 3950 60  0000 C CNN
 F 1 "PCM5100" H 5950 3400 60  0000 C CNN
 F 2 "" H 4250 5300 60  0000 C CNN
@@
 $EndComp
 $Comp
-L +3.3V #PWR?
+L +3.3V #PWR503
 U 1 1 53676BDD
 P 5650 2100
-F 0 "#PWR?" H 5650 2060 30  0001 C CNN
+F 0 "#PWR503" H 5650 2060 30  0001 C CNN
 F 1 "+3.3V" H 5650 2210 30  0000 C CNN
 F 2 "" H 5650 2100 60  0000 C CNN
@@
 Connection ~ 5900 2150
 $Comp
-L CPSMALL C?
+L CPSMALL C504
 U 1 1 53676C04
 P 5500 2300
-F 0 "C?" H 5525 2350 30  0000 L CNN
+F 0 "C504" H 5525 2350 30  0000 L CNN
 F 1 "10uF" H 5525 2225 30  0000 L CNN
 F 2 "~" H 5500 2300 60  0000 C CNN
@@
 $EndComp
 $Comp
-L CSMALL C?
+L CSMALL C503
 U 1 1 53676C1F
 P 5200 2300
-F 0 "C?" H 5225 2350 30  0000 L CNN
+F 0 "C503" H 5225 2350 30  0000 L CNN
 F 1 "100nF" H 5225 2250 30  0000 L CNN
 F 2 "~" H 5200 2300 60  0000 C CNN
@@
 $EndComp
 $Comp
-L CSMALL C?
+L CSMALL C502
 U 1 1 53676C42
 P 4950 2300
-F 0 "C?" H 4975 2350 30  0000 L CNN
+F 0 "C502" H 4975 2350 30  0000 L CNN
 F 1 "100nF" H 4975 2250 30  0000 L CNN
 F 2 "~" H 4950 2300 60  0000 C CNN
@@
 $EndComp
 $Comp
-L CSMALL C?
+L CSMALL C501
 U 1 1 53676C48
 P 4700 2300
-F 0 "C?" H 4725 2350 30  0000 L CNN
+F 0 "C501" H 4725 2350 30  0000 L CNN
 F 1 "100nF" H 4725 2250 30  0000 L CNN
 F 2 "~" H 4700 2300 60  0000 C CNN
@@
 Connection ~ 5500 2150
 $Comp
-L GND #PWR?
+L GND #PWR501
 U 1 1 53676C8D
 P 5100 2500
-F 0 "#PWR?" H 5100 2500 30  0001 C CNN
+F 0 "#PWR501" H 5100 2500 30  0001 C CNN
 F 1 "GND" H 5100 2430 30  0001 C CNN
 F 2 "" H 5100 2500 60  0000 C CNN
@@
 Connection ~ 5200 2450
 $Comp
-L GND #PWR?
+L GND #PWR504
 U 1 1 53676F41
 P 5950 4300
-F 0 "#PWR?" H 5950 4300 30  0001 C CNN
+F 0 "#PWR504" H 5950 4300 30  0001 C CNN
 F 1 "GND" H 5950 4230 30  0001 C CNN
 F 2 "" H 5950 4300 60  0000 C CNN
@@
 OUTL
 $Comp
-L R R?
+L R R501
 U 1 1 53676FA8
 P 7050 3000
-F 0 "R?" V 7130 3000 40  0000 C CNN
+F 0 "R501" V 7130 3000 40  0000 C CNN
 F 1 "470" V 7057 3001 40  0000 C CNN
 F 2 "~" V 6980 3000 30  0000 C CNN
@@
 $EndComp
 $Comp
-L R R?
+L R R502
 U 1 1 53676FD0
 P 7400 3100
-F 0 "R?" V 7480 3100 40  0000 C CNN
+F 0 "R502" V 7480 3100 40  0000 C CNN
 F 1 "470" V 7407 3101 40  0000 C CNN
 F 2 "~" V 7330 3100 30  0000 C CNN
@@
 $EndComp
 $Comp
-L C C?
+L C C508
 U 1 1 53676FE9
 P 7850 3350
-F 0 "C?" H 7850 3450 40  0000 L CNN
+F 0 "C508" H 7850 3450 40  0000 L CNN
 F 1 "2.2nF" H 7856 3265 40  0000 L CNN
 F 2 "~" H 7888 3200 30  0000 C CNN
@@
 $EndComp
 $Comp
-L C C?
+L C C509
 U 1 1 53676FFB
 P 8050 3350
-F 0 "C?" H 8050 3450 40  0000 L CNN
+F 0 "C509" H 8050 3450 40  0000 L CNN
 F 1 "2.2nF" H 8056 3265 40  0000 L CNN
 F 2 "~" H 8088 3200 30  0000 C CNN
@@
 Connection ~ 7850 3100
 $Comp
-L GND #PWR?
+L GND #PWR506
 U 1 1 536770C1
 P 7850 3600
-F 0 "#PWR?" H 7850 3600 30  0001 C CNN
+F 0 "#PWR506" H 7850 3600 30  0001 C CNN
 F 1 "GND" H 7850 3530 30  0001 C CNN
 F 2 "" H 7850 3600 60  0000 C CNN
@@
 $EndComp
 $Comp
-L GND #PWR?
+L GND #PWR507
 U 1 1 536770D1
 P 8050 3600
-F 0 "#PWR?" H 8050 3600 30  0001 C CNN
+F 0 "#PWR507" H 8050 3600 30  0001 C CNN
 F 1 "GND" H 8050 3530 30  0001 C CNN
 F 2 "" H 8050 3600 60  0000 C CNN
@@
 	7850 3600 7850 3550
 $Comp
-L CPSMALL C?
+L CPSMALL C506
 U 1 1 536775E2
 P 7000 3400
-F 0 "C?" H 7025 3450 30  0000 L CNN
+F 0 "C506" H 7025 3450 30  0000 L CNN
 F 1 "2.2uF" H 7025 3325 30  0000 L CNN
 F 2 "~" H 7000 3400 60  0000 C CNN
@@
 	6750 3500 7000 3500
 $Comp
-L CPSMALL C?
+L CPSMALL C507
 U 1 1 5367765A
 P 7200 3600
-F 0 "C?" H 7225 3650 30  0000 L CNN
+F 0 "C507" H 7225 3650 30  0000 L CNN
 F 1 "2.2uF" H 7225 3525 30  0000 L CNN
 F 2 "~" H 7200 3600 60  0000 C CNN
@@
 $EndComp
 $Comp
-L GND #PWR?
+L GND #PWR505
 U 1 1 5367766A
 P 7450 4000
-F 0 "#PWR?" H 7450 4000 30  0001 C CNN
+F 0 "#PWR505" H 7450 4000 30  0001 C CNN
 F 1 "GND" H 7450 3930 30  0001 C CNN
 F 2 "" H 7450 4000 60  0000 C CNN
@@
 	7100 3600 6750 3600
 $Comp
-L CSMALL C?
+L CSMALL C505
 U 1 1 536776D6
 P 6800 3850
-F 0 "C?" H 6825 3900 30  0000 L CNN
+F 0 "C505" H 6825 3900 30  0000 L CNN
 F 1 "100nF" H 6825 3800 30  0000 L CNN
 F 2 "~" H 6800 3850 60  0000 C CNN
@@
 	6800 3700 6750 3700
 $Comp
-L GND #PWR?
+L GND #PWR502
 U 1 1 536779A6
 P 5100 3950
-F 0 "#PWR?" H 5100 3950 30  0001 C CNN
+F 0 "#PWR502" H 5100 3950 30  0001 C CNN
 F 1 "GND" H 5100 3880 30  0001 C CNN
 F 2 "" H 5100 3950 60  0000 C CNN
