File: kicad/project one mpu.sch (KiCad schematic (older format))
At the start: 28 parts, among them J301 USB, J302 5P HDR, SW301 DFU, SW302 RESET, U301 AT32UC3C1512C, U302 AT24C32, U303 CS2200-CP, X301 12 MHz

Commit message: ..more work
Parts:
- added R?: 330, ~, symbol R
Connections:
- net labels added: ADC_OVF, AUDIO_RESET, DAC_FLT, DAC_XSMT
- wire segments 121 -> 166
Other:
- moved on the sheet: R304, SW302
Changed lines of the file:
@@
 $Descr USLetter 11000 8500
 encoding utf-8
-Sheet 3 4
+Sheet 3 6
 Title "Project One"
-Date "4 may 2014"
+Date "5 may 2014"
 Rev "0.0.0"
 Comp "Ali Kocaturk"
@@
 L +3.3V #PWR306
 U 1 1 536676CF
-P 2450 6750
-F 0 "#PWR306" H 2450 6710 30  0001 C CNN
-F 1 "+3.3V" H 2450 6860 30  0000 C CNN
-F 2 "" H 2450 6750 60  0000 C CNN
-F 3 "" H 2450 6750 60  0000 C CNN
-	1    2450 6750
+P 2100 6750
+F 0 "#PWR306" H 2100 6710 30  0001 C CNN
+F 1 "+3.3V" H 2100 6860 30  0000 C CNN
+F 2 "" H 2100 6750 60  0000 C CNN
+F 3 "" H 2100 6750 60  0000 C CNN
+	1    2100 6750
 	1    0    0    -1
 $EndComp
@@
 L SW_PUSH SW302
 U 1 1 536676E2
-P 3050 7200
-F 0 "SW302" H 3200 7310 50  0000 C CNN
-F 1 "RESET" H 3050 7120 50  0000 C CNN
-F 2 "~" H 3050 7200 60  0000 C CNN
-F 3 "~" H 3050 7200 60  0000 C CNN
-	1    3050 7200
+P 2750 7200
+F 0 "SW302" H 2900 7310 50  0000 C CNN
+F 1 "RESET" H 2750 7120 50  0000 C CNN
+F 2 "~" H 2750 7200 60  0000 C CNN
+F 3 "~" H 2750 7200 60  0000 C CNN
+	1    2750 7200
 	0    -1   -1   0
 $EndComp
@@
 L GND #PWR307
 U 1 1 536676E8
-P 3050 7600
-F 0 "#PWR307" H 3050 7600 30  0001 C CNN
-F 1 "GND" H 3050 7530 30  0001 C CNN
-F 2 "" H 3050 7600 60  0000 C CNN
-F 3 "" H 3050 7600 60  0000 C CNN
-	1    3050 7600
+P 2750 7600
+F 0 "#PWR307" H 2750 7600 30  0001 C CNN
+F 1 "GND" H 2750 7530 30  0001 C CNN
+F 2 "" H 2750 7600 60  0000 C CNN
+F 3 "" H 2750 7600 60  0000 C CNN
+	1    2750 7600
 	1    0    0    -1
 $EndComp
@@
 L R R304
 U 1 1 536676EF
-P 2750 6800
-F 0 "R304" V 2830 6800 40  0000 C CNN
-F 1 "10k" V 2757 6801 40  0000 C CNN
-F 2 "~" V 2680 6800 30  0000 C CNN
-F 3 "~" H 2750 6800 30  0000 C CNN
-	1    2750 6800
+P 2450 6800
+F 0 "R304" V 2530 6800 40  0000 C CNN
+F 1 "10k" V 2457 6801 40  0000 C CNN
+F 2 "~" V 2380 6800 30  0000 C CNN
+F 3 "~" H 2450 6800 30  0000 C CNN
+	1    2450 6800
 	0    -1   -1   0
 $EndComp
@@
 	1600 1650 800  1650
 Wire Wire Line
-	800  1650 800  2250
+	800  1650 800  1900
+Wire Wire Line
+	800  1900 800  2000
+Wire Wire Line
+	800  2000 800  2250
 Wire Wire Line
 	800  1900 850  1900
@@
 Connection ~ 2200 1000
 Wire Wire Line
-	4600 1100 4600 1400
+	4600 1100 4600 1250
+Wire Wire Line
+	4600 1250 4600 1400
 Wire Wire Line
 	4600 1250 4650 1250
 Connection ~ 4600 1250
 Wire Wire Line
-	3050 7500 3050 7600
-Wire Wire Line
-	3050 6800 3050 6900
+	2750 7500 2750 7550
+Wire Wire Line
+	2750 7550 2750 7600
+Wire Wire Line
+	2750 6800 2750 6900
 Wire Wire Line
 	3350 7550 3350 7300
-Connection ~ 3050 7550
-Wire Wire Line
-	3000 6800 3350 6800
-Wire Wire Line
-	3350 6750 3350 7100
-Connection ~ 3050 6800
-Wire Wire Line
-	2450 6750 2450 6800
+Connection ~ 2750 7550
+Wire Wire Line
+	2700 6800 2750 6800
+Wire Wire Line
+	2750 6800 2800 6800
+Wire Wire Line
+	3350 6750 3350 6800
+Wire Wire Line
+	3350 6800 3350 7100
+Connection ~ 2750 6800
+Wire Wire Line
+	2100 6750 2100 6800
 Connection ~ 3350 6800
 Wire Wire Line
-	4050 7550 4050 6750
+	4050 7550 4050 6800
+Wire Wire Line
+	4050 6800 4050 6750
 Connection ~ 3350 7550
 Wire Wire Line
-	4050 6800 4550 6800
+	4050 6800 4150 6800
+Wire Wire Line
+	4150 6800 4250 6800
+Wire Wire Line
+	4250 6800 4350 6800
+Wire Wire Line
+	4350 6800 4450 6800
+Wire Wire Line
+	4450 6800 4550 6800
 Wire Wire Line
 	4150 6800 4150 6750
@@
 	5900 6050 7100 6050
 Wire Wire Line
-	1450 1000 4250 1000
+	1450 1000 1750 1000
+Wire Wire Line
+	1750 1000 2050 1000
+Wire Wire Line
+	2050 1000 2200 1000
+Wire Wire Line
+	2200 1000 2350 1000
+Wire Wire Line
+	2350 1000 2650 1000
+Wire Wire Line
+	2650 1000 3500 1000
+Wire Wire Line
+	3500 1000 3600 1000
+Wire Wire Line
+	3600 1000 3700 1000
+Wire Wire Line
+	3700 1000 3800 1000
+Wire Wire Line
+	3800 1000 4050 1000
+Wire Wire Line
+	4050 1000 4250 1000
 Wire Wire Line
 	1450 1000 1450 1050
@@
 	1450 1250 1450 1300
 Wire Wire Line
-	1450 1300 2650 1300
+	1450 1300 1750 1300
+Wire Wire Line
+	1750 1300 2050 1300
+Wire Wire Line
+	2050 1300 2200 1300
+Wire Wire Line
+	2200 1300 2350 1300
+Wire Wire Line
+	2350 1300 2650 1300
 Wire Wire Line
 	2050 1300 2050 1250
@@
 	7750 6350 8500 6350
 Wire Wire Line
-	9200 6750 9200 6850
-Wire Wire Line
-	9950 6800 8450 6800
-Wire Wire Line
-	9950 5700 9950 6800
+	9200 6750 9200 6800
+Wire Wire Line
+	9200 6800 9200 6850
+Wire Wire Line
+	9950 6800 9200 6800
+Wire Wire Line
+	9200 6800 8450 6800
+Wire Wire Line
+	9950 5700 9950 6050
+Wire Wire Line
+	9950 6050 9950 6150
+Wire Wire Line
+	9950 6150 9950 6250
+Wire Wire Line
+	9950 6250 9950 6800
 Wire Wire Line
 	9950 5700 9450 5700
@@
 Connection ~ 9950 6250
 Wire Wire Line
-	9200 5650 9200 5750
+	9200 5650 9200 5700
+Wire Wire Line
+	9200 5700 9200 5750
 Wire Wire Line
 	9200 5700 9250 5700
@@
 	8450 6150 8450 6800
 Wire Wire Line
-	6300 5500 6300 5650
+	6300 5500 6300 5550
+Wire Wire Line
+	6300 5550 6300 5650
 Wire Wire Line
 	6300 5550 6450 5550
 Connection ~ 6300 5550
 Wire Bus Line
-	7200 5500 7200 6050
+	7200 5500 7200 5950
+Wire Bus Line
+	7200 5950 7200 6050
 Wire Bus Line
 	7650 2800 8450 2800
 Wire Bus Line
-	7650 2800 7650 6350
+	7650 2800 7650 4100
+Wire Bus Line
+	7650 4100 7650 4200
+Wire Bus Line
+	7650 4200 7650 6250
+Wire Bus Line
+	7650 6250 7650 6350
 Wire Wire Line
 	6950 3550 5900 3550
@@
 	1150 3800 1200 3800
 Wire Wire Line
-	1700 3800 2300 3800
+	1700 3800 1750 3800
+Wire Wire Line
+	1750 3800 2300 3800
 Wire Wire Line
 	1750 3800 1750 3850
@@
 Connection ~ 1750 3800
 Wire Wire Line
-	2450 6800 2500 6800
-Wire Wire Line
-	3050 7550 5200 7550
-Wire Wire Line
-	7850 4450 7850 4750
+	2100 6800 2200 6800
+Wire Wire Line
+	2750 7550 3350 7550
+Wire Wire Line
+	3350 7550 4050 7550
+Wire Wire Line
+	4050 7550 4900 7550
+Wire Wire Line
+	4900 7550 5200 7550
+Wire Wire Line
+	7850 4450 7850 4700
+Wire Wire Line
+	7850 4700 7850 4750
 Wire Wire Line
 	7850 4700 7900 4700
@@
 	7850 4450 8550 4450
 Wire Wire Line
-	8550 4550 8550 4750
+	8550 4550 8550 4700
+Wire Wire Line
+	8550 4700 8550 4750
 Wire Wire Line
 	8500 4700 8550 4700
 Connection ~ 8550 4700
 Wire Wire Line
-	9600 4950 9600 5250
-Wire Wire Line
-	7850 5200 9700 5200
+	9600 4950 9600 5200
+Wire Wire Line
+	9600 5200 9600 5250
+Wire Wire Line
+	7850 5200 8550 5200
+Wire Wire Line
+	8550 5200 9600 5200
+Wire Wire Line
+	9600 5200 9700 5200
 Wire Wire Line
 	9700 5200 9700 4950
@@
 	8750 3600 8750 3550
 Wire Wire Line
-	8500 3550 9000 3550
+	8500 3550 8750 3550
+Wire Wire Line
+	8750 3550 9000 3550
 Wire Wire Line
 	8500 3550 8500 4200
@@
 $EndComp
 Wire Wire Line
-	9400 3500 9400 3600
+	9400 3500 9400 3550
+Wire Wire Line
+	9400 3550 9400 3600
 Wire Wire Line
 	9400 3550 9200 3550
@@
 	1350 5400 1750 5400
 Wire Bus Line
-	1750 5400 1750 6000
+	1750 5400 1750 5600
+Wire Bus Line
+	1750 5600 1750 5700
+Wire Bus Line
+	1750 5700 1750 5800
+Wire Bus Line
+	1750 5800 1750 5900
+Wire Bus Line
+	1750 5900 1750 6000
 Text Label 10450 4000 2    60   ~ 0
 XIN1
@@
 Connection ~ 4050 1000
 Wire Wire Line
-	4900 1400 4900 1100
+	4900 1100 4900 1250
+Wire Wire Line
+	4900 1250 4900 1400
 Wire Wire Line
 	4900 1100 4850 1100
@@
 Wire Bus Line
 	7200 5500 7650 5500
+Text HLabel 8050 1550 2    60   Input ~ 0
+ADC_OVF
+Text HLabel 8050 1700 2    60   Output ~ 0
+AUDIO_RESET
+Text HLabel 9950 1600 0    60   Output ~ 0
+DAC_XSMT
+Text HLabel 9950 1700 0    60   Output ~ 0
+DAC_FLT
+$Comp
+L R R?
+U 1 1 5367423B
+P 3050 6800
+F 0 "R?" V 3130 6800 40  0000 C CNN
+F 1 "330" V 3057 6801 40  0000 C CNN
+F 2 "~" V 2980 6800 30  0000 C CNN
+F 3 "~" H 3050 6800 30  0000 C CNN
+	1    3050 6800
+	0    -1   -1   0
+$EndComp
+Wire Wire Line
+	3350 6800 3300 6800
 $EndSCHEMATC

Commit message: Work on amplifier sheeet
Connections:
- wire segments 166 -> 122
Other:
- note added: "Hierarchial pins\n(to be wired)"
Changed lines of the file:
@@
 	1600 1650 800  1650
 Wire Wire Line
-	800  1650 800  1900
-Wire Wire Line
-	800  1900 800  2000
-Wire Wire Line
-	800  2000 800  2250
+	800  1650 800  2250
 Wire Wire Line
 	800  1900 850  1900
@@
 Connection ~ 2200 1000
 Wire Wire Line
-	4600 1100 4600 1250
-Wire Wire Line
-	4600 1250 4600 1400
+	4600 1100 4600 1400
 Wire Wire Line
 	4600 1250 4650 1250
 Connection ~ 4600 1250
 Wire Wire Line
-	2750 7500 2750 7550
-Wire Wire Line
-	2750 7550 2750 7600
+	2750 7500 2750 7600
 Wire Wire Line
 	2750 6800 2750 6900
@@
 Connection ~ 2750 7550
 Wire Wire Line
-	2700 6800 2750 6800
-Wire Wire Line
-	2750 6800 2800 6800
-Wire Wire Line
-	3350 6750 3350 6800
-Wire Wire Line
-	3350 6800 3350 7100
+	2700 6800 2800 6800
+Wire Wire Line
+	3350 6750 3350 7100
 Connection ~ 2750 6800
 Wire Wire Line
@@
 Connection ~ 3350 6800
 Wire Wire Line
-	4050 7550 4050 6800
-Wire Wire Line
-	4050 6800 4050 6750
+	4050 7550 4050 6750
 Connection ~ 3350 7550
 Wire Wire Line
-	4050 6800 4150 6800
-Wire Wire Line
-	4150 6800 4250 6800
-Wire Wire Line
-	4250 6800 4350 6800
-Wire Wire Line
-	4350 6800 4450 6800
-Wire Wire Line
-	4450 6800 4550 6800
+	4050 6800 4550 6800
 Wire Wire Line
 	4150 6800 4150 6750
@@
 	5900 6050 7100 6050
 Wire Wire Line
-	1450 1000 1750 1000
-Wire Wire Line
-	1750 1000 2050 1000
-Wire Wire Line
-	2050 1000 2200 1000
-Wire Wire Line
-	2200 1000 2350 1000
-Wire Wire Line
-	2350 1000 2650 1000
-Wire Wire Line
-	2650 1000 3500 1000
-Wire Wire Line
-	3500 1000 3600 1000
-Wire Wire Line
-	3600 1000 3700 1000
-Wire Wire Line
-	3700 1000 3800 1000
-Wire Wire Line
-	3800 1000 4050 1000
-Wire Wire Line
-	4050 1000 4250 1000
+	1450 1000 4250 1000
 Wire Wire Line
 	1450 1000 1450 1050
@@
 	1450 1250 1450 1300
 Wire Wire Line
-	1450 1300 1750 1300
-Wire Wire Line
-	1750 1300 2050 1300
-Wire Wire Line
-	2050 1300 2200 1300
-Wire Wire Line
-	2200 1300 2350 1300
-Wire Wire Line
-	2350 1300 2650 1300
+	1450 1300 2650 1300
 Wire Wire Line
 	2050 1300 2050 1250
@@
 	7750 6350 8500 6350
 Wire Wire Line
-	9200 6750 9200 6800
-Wire Wire Line
-	9200 6800 9200 6850
-Wire Wire Line
-	9950 6800 9200 6800
-Wire Wire Line
-	9200 6800 8450 6800
-Wire Wire Line
-	9950 5700 9950 6050
-Wire Wire Line
-	9950 6050 9950 6150
-Wire Wire Line
-	9950 6150 9950 6250
-Wire Wire Line
-	9950 6250 9950 6800
+	9200 6750 9200 6850
+Wire Wire Line
+	9950 6800 8450 6800
+Wire Wire Line
+	9950 5700 9950 6800
 Wire Wire Line
 	9950 5700 9450 5700
@@
 Connection ~ 9950 6250
 Wire Wire Line
-	9200 5650 9200 5700
-Wire Wire Line
-	9200 5700 9200 5750
+	9200 5650 9200 5750
 Wire Wire Line
 	9200 5700 9250 5700
@@
 	8450 6150 8450 6800
 Wire Wire Line
-	6300 5500 6300 5550
-Wire Wire Line
-	6300 5550 6300 5650
+	6300 5500 6300 5650
 Wire Wire Line
 	6300 5550 6450 5550
 Connection ~ 6300 5550
 Wire Bus Line
-	7200 5500 7200 5950
-Wire Bus Line
-	7200 5950 7200 6050
+	7200 5500 7200 6050
 Wire Bus Line
 	7650 2800 8450 2800
 Wire Bus Line
-	7650 2800 7650 4100
-Wire Bus Line
-	7650 4100 7650 4200
-Wire Bus Line
-	7650 4200 7650 6250
-Wire Bus Line
-	7650 6250 7650 6350
+	7650 2800 7650 6350
 Wire Wire Line
 	6950 3550 5900 3550
@@
 	1150 3800 1200 3800
 Wire Wire Line
-	1700 3800 1750 3800
-Wire Wire Line
-	1750 3800 2300 3800
+	1700 3800 2300 3800
 Wire Wire Line
 	1750 3800 1750 3850
@@
 	2100 6800 2200 6800
 Wire Wire Line
-	2750 7550 3350 7550
-Wire Wire Line
-	3350 7550 4050 7550
-Wire Wire Line
-	4050 7550 4900 7550
-Wire Wire Line
-	4900 7550 5200 7550
-Wire Wire Line
-	7850 4450 7850 4700
-Wire Wire Line
-	7850 4700 7850 4750
+	2750 7550 5200 7550
+Wire Wire Line
+	7850 4450 7850 4750
 Wire Wire Line
 	7850 4700 7900 4700
@@
 	7850 4450 8550 4450
 Wire Wire Line
-	8550 4550 8550 4700
-Wire Wire Line
-	8550 4700 8550 4750
+	8550 4550 8550 4750
 Wire Wire Line
 	8500 4700 8550 4700
 Connection ~ 8550 4700
 Wire Wire Line
-	9600 4950 9600 5200
-Wire Wire Line
-	9600 5200 9600 5250
-Wire Wire Line
-	7850 5200 8550 5200
-Wire Wire Line
-	8550 5200 9600 5200
-Wire Wire Line
-	9600 5200 9700 5200
+	9600 4950 9600 5250
+Wire Wire Line
+	7850 5200 9700 5200
 Wire Wire Line
 	9700 5200 9700 4950
@@
 	8750 3600 8750 3550
 Wire Wire Line
-	8500 3550 8750 3550
-Wire Wire Line
-	8750 3550 9000 3550
+	8500 3550 9000 3550
 Wire Wire Line
 	8500 3550 8500 4200
@@
 $EndComp
 Wire Wire Line
-	9400 3500 9400 3550
-Wire Wire Line
-	9400 3550 9400 3600
+	9400 3500 9400 3600
 Wire Wire Line
 	9400 3550 9200 3550
@@
 	1350 5400 1750 5400
 Wire Bus Line
-	1750 5400 1750 5600
-Wire Bus Line
-	1750 5600 1750 5700
-Wire Bus Line
-	1750 5700 1750 5800
-Wire Bus Line
-	1750 5800 1750 5900
-Wire Bus Line
-	1750 5900 1750 6000
+	1750 5400 1750 6000
 Text Label 10450 4000 2    60   ~ 0
 XIN1
@@
 Connection ~ 4050 1000
 Wire Wire Line
-	4900 1100 4900 1250
-Wire Wire Line
-	4900 1250 4900 1400
+	4900 1100 4900 1400
 Wire Wire Line
 	4900 1100 4850 1100
@@
 Wire Wire Line
 	3350 6800 3300 6800
+Wire Notes Line
+	7750 1150 7750 2250
+Wire Notes Line
+	7750 2250 10300 2250
+Wire Notes Line
+	10300 2250 10300 1200
+Wire Notes Line
+	10300 1200 7750 1200
+Text Notes 8700 1100 0    60   ~ 0
+Hierarchial pins\n(to be wired)
 $EndSCHEMATC

Commit message: Forgot to add annotation
Parts:
- gave numbers to parts that had none: 1
- renumbered R305 to R306, R306 to R307
Changed lines of the file:
@@
 $EndComp
 $Comp
-L +3.3V #PWR304
+L +3.3V #PWR305
 U 1 1 5365F3C9
 P 2200 950
-F 0 "#PWR304" H 2200 910 30  0001 C CNN
+F 0 "#PWR305" H 2200 910 30  0001 C CNN
 F 1 "+3.3V" H 2200 1060 30  0000 C CNN
 F 2 "" H 2200 950 60  0000 C CNN
@@
 $EndComp
 $Comp
-L GND #PWR305
+L GND #PWR306
 U 1 1 5365F3F8
 P 2200 1350
-F 0 "#PWR305" H 2200 1350 30  0001 C CNN
+F 0 "#PWR306" H 2200 1350 30  0001 C CNN
 F 1 "GND" H 2200 1280 30  0001 C CNN
 F 2 "" H 2200 1350 60  0000 C CNN
@@
 $EndComp
 $Comp
-L +3.3V #PWR306
+L +3.3V #PWR304
 U 1 1 536676CF
 P 2100 6750
-F 0 "#PWR306" H 2100 6710 30  0001 C CNN
+F 0 "#PWR304" H 2100 6710 30  0001 C CNN
 F 1 "+3.3V" H 2100 6860 30  0000 C CNN
 F 2 "" H 2100 6750 60  0000 C CNN
@@
 TWIMS0
 $Comp
-L R R306
+L R R307
 U 1 1 53668F62
 P 6450 5800
-F 0 "R306" V 6530 5800 40  0000 C CNN
+F 0 "R307" V 6530 5800 40  0000 C CNN
 F 1 "4.7k" V 6457 5801 40  0000 C CNN
 F 2 "~" V 6380 5800 30  0000 C CNN
@@
 $EndComp
 $Comp
-L R R305
+L R R306
 U 1 1 53668F7A
 P 6300 5900
-F 0 "R305" V 6380 5900 40  0000 C CNN
+F 0 "R306" V 6380 5900 40  0000 C CNN
 F 1 "4.7k" V 6307 5901 40  0000 C CNN
 F 2 "~" V 6230 5900 30  0000 C CNN
@@
 DAC_FLT
 $Comp
-L R R?
+L R R305
 U 1 1 5367423B
 P 3050 6800
-F 0 "R?" V 3130 6800 40  0000 C CNN
+F 0 "R305" V 3130 6800 40  0000 C CNN
 F 1 "330" V 3057 6801 40  0000 C CNN
 F 2 "~" V 2980 6800 30  0000 C CNN

Commit message: More stuff....
Parts:
- added J?: 5x2P HDR, symbol CONN_5X2
- added U?: TSOP4838, symbol CONN_3
Connections:
- net labels added: AMP_DR_MUTE, AMP_HP_DETECT, AMP_SPK_FAULT, AMP_SPK_SD, QDEC0_QEPA, QDEC0_QEPB, QDEC1_QEPA, QDEC1_QEPB, TC0_B2
- wire segments 122 -> 132
Other:
- note added: "ENCODERS"
- moved on the sheet: R306, R307
