File: kicad/project one power supplies.sch (KiCad schematic (older format))
At the start: 25 parts

Commit message: More work on schematic
Parts:
- removed C?: 10uF, ~, symbol CAPAPOL
- removed L?: 2.2uH, ~, symbol INDUCTOR_SMALL
- removed R?: 33k, ~, symbol R
- removed R?: 10k, ~, symbol R
- removed U?: LM3671, symbol LM3671
- added C207: 22uF, ~, symbol CAPAPOL
- added D201: PWR_12V, ~, symbol LED
- added D202: PWR_5VA, ~, symbol LED
- added D203: PWR_3V3, ~, symbol LED
- added D207: PWR_5VD, ~, symbol LED
- added R201: 1.2k 1/4W, ~, symbol R
- added R202, R208: 330, ~, symbol R
- added R203: 150, ~, symbol R
- added U202: LMS8117ADT-3.3, TO-252, symbol LM1084IT-3.3/NOPB
- gave numbers to parts that had none: 20
Connections:
- wire segments 62 -> 64
Other:
- note added: "12V IN"
- moved on the sheet: C204
