File: kicad/main board/prj-one-mainboard.sch (KiCad schematic (older format))
At the start: 84 parts

Commit message: Switch to op-amp based design
Parts:
- removed C? (x6): 47u, ~, symbol CAPAPOL
- removed C? (x12): 1u, ~, symbol CAPAPOL
- removed Q? (x6): NPN, ~, symbol NPN
- removed R? (x6): 2.2k, ~, symbol R
- removed R? (x6): 10k, ~, symbol R
- removed R? (x6): 470k, ~, symbol R
- removed R? (x6): 100k, ~, symbol R
- removed R? (x18): 22k, ~, symbol R
- removed R? (x6): 220k, ~, symbol R
- removed RV? (x6): 100k, ~, symbol POT
- removed SW?: IN1_MUTE, ~, symbol DPST
- removed SW?: IN2_MUTE, ~, symbol DPST
- removed SW?: IN3_MUTE, ~, symbol DPST
- removed U?: TL082, symbol TL082
- added C?: 100u, ~, symbol CAPAPOL
- added R? (x2): 10k, ~, symbol R
- added U101: LM7812, ~, symbol LM7812
- added U103: LM1875, TO220-5, symbol LM1875
- added U?: TL072, symbol TL072
- K102: renamed from K?; value AIN1 -> AUDIO_IN
- gave numbers to parts that had none: 1
Connections:
- net labels added: +12V, 12V/2, L_MIX_OUT
- net labels removed: AGN1_L, AGN1_R, AGN2_L, AGN2_R, AGN3_L, AGN3_R, AIN1_L, AIN1_R, AIN2_L, AIN2_R, AIN3_L, AIN3_R, MIX_L, MIX_R
- wire segments 188 -> 21
Other:
- note removed: "GAIN1_L"
- note removed: "GAIN1_R"
- note removed: "GAIN2_L"
- note removed: "GAIN2_R"
- note removed: "GAIN3_L"
- note removed: "GAIN3_R"
- note removed: "Level Adjuster"
- moved on the sheet: K101, K102

Commit message: Simplify mixer design, remove power amp
Parts:
- removed K101: PWR, symbol CONN_2
- removed K102: AUDIO_IN, symbol CONN_3
- removed U103: LM1875, TO220-5, symbol LM1875
- removed U?: TL072, symbol TL072
- added BASS1, BASS2, TREB1, TREB2, VOL1, VOL2: 100k, ~, symbol POT
- added C1, C14, C15, C16, C17, C5, C6: 100n, ~, symbol C
- added C10, C13, C18, C2, C22, C25, C26, C27: 100p, ~, symbol C
- added C11, C23: 47n, ~, symbol C
- added C12, C24: 1n, ~, symbol C
- added C19, C20, C28, C29, C3, C7, C8: 10u, ~, symbol CAPAPOL
- added C21, C4: 100u, ~, symbol CAPAPOL
- added H1, H2, H3, H4: CONN_1, symbol CONN_1
- added J1, J2, J3, J4, J5: JACK_6P, ~, symbol JACK_6P
- added J6: PJ-037, ~, symbol PJ-037
- added R1, R14, R22, R27, R35, R43, R44, R6: 2.2k, ~, symbol R
- added R10, R12, R17, R20, R21, R24, R3, R31, R33, R38, R41, R42, R45, R46: 22k, ~, symbol R
- added R11, R32: 150k, ~, symbol R
- added R13, R16, R18, R26, R30, R34, R37, R39: 10k, ~, symbol R
- added R15, R19, R2, R23, R28, R36, R40, R7: 470k, ~, symbol R
- added R25, R4: 1M, ~, symbol R
- added R29, R8: 15k, ~, symbol R
- added TONE1, TONE2: TONE, ~, symbol SWITCH_INV
- added U1: TL072, symbol TL072
- added U2: TL074, symbol TL074
- gave numbers to parts that had none: 3
- renumbered U101 to U3
Connections:
- net labels added: LIN1_L, LIN1_R, LIN2_L, LIN2_R, LIN3_L, LIN3_R, LIN4_L, LIN4_R, PREOUT_L, PREOUT_R
- net labels removed: L_MIX_OUT, VCC
- wire segments 21 -> 244
- no-connect marks 0 -> 2
Other:
- moved on the sheet: C9, R5, R9, U3
